Commit message: 发现问题

File: source/robot_lab/data/Robots/unitree/a1_description/urdf/a1.urdf (robot description, URDF)
Before this commit: robot a1, 23 links, 22 joints
Links:
- removed link FL_thigh_shoulder
- removed link FR_thigh_shoulder
- removed link RL_thigh_shoulder
- removed link RR_thigh_shoulder
- removed link imu_link
- added link FL_calflower; collision box size=0.05 0.0258 0.025
- added link FL_calflower1; collision box size=0.05 0.0258 0.025
- added link FR_calflower; collision box size=0.05 0.0258 0.025
- added link FR_calflower1; collision box size=0.05 0.0258 0.025
- added link RL_calflower; collision box size=0.05 0.0258 0.025
- added link RL_calflower1; collision box size=0.05 0.0258 0.025
- added link RR_calflower; collision box size=0.05 0.0258 0.025
- added link RR_calflower1; collision box size=0.05 0.0258 0.025
- added link base_imu, mass 0.01; visual box size=0.015 0.015 0.004
- link FL_calf: mass 0.166 -> 0.1304; geometry collision box size=0.1067 0.02988 0.024; visual mesh filename=../meshes/calf.dae scale=1 1 1
- link FL_foot: mass 0.06 -> 0.0311609; geometry collision sphere radius=0.021; visual sphere radius=0.011000000000000001
- link FL_hip: mass 0.696 -> 0.9754; geometry collision cylinder length=0.0631 radius=0.06275; visual mesh filename=../meshes/hip.dae scale=1 1 1
- link FL_thigh: mass 1.013 -> 1.6868; geometry collision box size=0.25 0.065 0.085; collision cylinder length=0.0655 radius=0.054
- link FR_calf: mass 0.166 -> 0.1304; geometry collision box size=0.1067 0.02988 0.024; visual mesh filename=../meshes/calf_mirror.dae scale=1 1 1
- link FR_foot: mass 0.06 -> 0.0911609; geometry collision sphere radius=0.021; visual sphere radius=0.011000000000000001
- link FR_hip: mass 0.696 -> 0.9754; geometry collision cylinder length=0.0631 radius=0.06275; visual mesh filename=../meshes/hip.dae scale=1 1 1
- link FR_thigh: mass 1.013 -> 1.6868; geometry collision box size=0.25 0.065 0.085; collision cylinder length=0.0655 radius=0.054
- link RL_calf: mass 0.166 -> 0.1304; geometry collision box size=0.1067 0.02988 0.024; visual mesh filename=../meshes/calf.dae scale=1 1 1
- link RL_foot: mass 0.06 -> 0.0911609; geometry collision sphere radius=0.021; visual sphere radius=0.011000000000000001
- link RL_hip: mass 0.696 -> 0.9754; geometry collision cylinder length=0.0631 radius=0.06275; visual mesh filename=../meshes/hip.dae scale=1 1 1
- link RL_thigh: mass 1.013 -> 1.6868; geometry collision box size=0.25 0.065 0.085; collision cylinder length=0.0655 radius=0.054
- link RR_calf: mass 0.166 -> 0.1304; geometry collision box size=0.1067 0.02988 0.024; visual mesh filename=../meshes/calf_mirror.dae scale=1 1 1
- link RR_foot: mass 0.06 -> 0.0911609; geometry collision sphere radius=0.021; visual sphere radius=0.011000000000000001
- link RR_hip: mass 0.696 -> 0.9754; geometry collision cylinder length=0.0631 radius=0.06275; visual mesh filename=../meshes/hip.dae scale=1 1 1
- link RR_thigh: mass 1.013 -> 1.6868; geometry collision box size=0.25 0.065 0.085; collision cylinder length=0.0655 radius=0.054
- link trunk: mass 6.0 -> 8.1152; geometry collision box size=0.32 0.252 0.135; visual mesh filename=../meshes/trunk.dae scale=1 1 1
Joints:
- removed joint FL_hip_fixed
- removed joint FR_hip_fixed
- removed joint RL_hip_fixed
- removed joint RR_hip_fixed
- removed joint imu_joint
- added joint FL_calflower1_joint: type fixed, parent FL_calflower, child FL_calflower1, origin xyz=0.03 0 -0.09 rpy=0 1.707963267948966 0, axis 0 0 0
- added joint FL_calflower_joint: type fixed, parent FL_calf, child FL_calflower, origin xyz=0 0 -0.1 rpy=0 0 0
- added joint FR_calflower1_joint: type fixed, parent FR_calflower, child FR_calflower1, origin xyz=0.03 0 -0.09 rpy=0 1.707963267948966 0, axis 0 0 0
- added joint FR_calflower_joint: type fixed, parent FR_calf, child FR_calflower, origin xyz=0 0 -0.1 rpy=0 0 0
- added joint RL_calflower1_joint: type fixed, parent RL_calflower, child RL_calflower1, origin xyz=0.03 0 -0.09 rpy=0 1.707963267948966 0, axis 0 0 0
- added joint RL_calflower_joint: type fixed, parent RL_calf, child RL_calflower, origin xyz=0 0 -0.1 rpy=0 0 0
- added joint RR_calflower1_joint: type fixed, parent RR_calflower, child RR_calflower1, origin xyz=0.03 0 -0.09 rpy=0 1.707963267948966 0, axis 0 0 0
- added joint RR_calflower_joint: type fixed, parent RR_calf, child RR_calflower, origin xyz=0 0 -0.1 rpy=0 0 0
- added joint base_imu_joint: type fixed, parent trunk, child base_imu, origin xyz=0. 0. 0. rpy=0. 0. 0.
- joint FL_calf_joint: limit lower=-2.69653369433 upper=-0.916297857297 effort=33.5 velocity=21 -> lower=-2.8012534494508987 upper=-0.7417649320975901 effort=53.5 velocity=11; origin xyz=0 0 -0.2 rpy=0 0 0 -> xyz=0 0 -0.25 rpy=0 0 0
- joint FL_foot_fixed: origin xyz=0 0 -0.2 rpy=0 0 0 -> xyz=0.01 0 -0.2287 rpy=0 0 0
- joint FL_hip_joint: limit lower=-0.802851455917 upper=0.802851455917 effort=33.5 velocity=21 -> lower=-0.9773843811168246 upper=0.9773843811168246 effort=53.5 velocity=11; origin xyz=0.1805 0.047 0 rpy=0 0 0 -> xyz=0.2305 0.055 0.01 rpy=0 0 0
- joint FL_thigh_joint: limit lower=-1.0471975512 upper=4.18879020479 effort=33.5 velocity=21 -> lower=-1.0471975511965976 upper=4.1887902047863905 effort=53.5 velocity=11; origin xyz=0 0.0838 0 rpy=0 0 0 -> xyz=0 0.1231 0 rpy=0 0 0
- joint FR_calf_joint: limit lower=-2.69653369433 upper=-0.916297857297 effort=33.5 velocity=21 -> lower=-2.8012534494508987 upper=-0.7417649320975901 effort=53.5 velocity=11; origin xyz=0 0 -0.2 rpy=0 0 0 -> xyz=0 0 -0.25 rpy=0 0 0
- joint FR_foot_fixed: origin xyz=0 0 -0.2 rpy=0 0 0 -> xyz=0.01 0 -0.2287 rpy=0 0 0
- joint FR_hip_joint: limit lower=-0.802851455917 upper=0.802851455917 effort=33.5 velocity=21 -> lower=-0.9773843811168246 upper=0.9773843811168246 effort=53.5 velocity=11; origin xyz=0.1805 -0.047 0 rpy=0 0 0 -> xyz=0.2305 -0.055 0.01 rpy=0 0 0
- joint FR_thigh_joint: limit lower=-1.0471975512 upper=4.18879020479 effort=33.5 velocity=21 -> lower=-1.0471975511965976 upper=4.1887902047863905 effort=53.5 velocity=11; origin xyz=0 -0.0838 0 rpy=0 0 0 -> xyz=0 -0.1231 0 rpy=0 0 0
- joint RL_calf_joint: limit lower=-2.69653369433 upper=-0.916297857297 effort=33.5 velocity=21 -> lower=-2.8012534494508987 upper=-0.7417649320975901 effort=53.5 velocity=11; origin xyz=0 0 -0.2 rpy=0 0 0 -> xyz=0 0 -0.25 rpy=0 0 0
- joint RL_foot_fixed: origin xyz=0 0 -0.2 rpy=0 0 0 -> xyz=0.01 0 -0.2287 rpy=0 0 0
- joint RL_hip_joint: limit lower=-0.802851455917 upper=0.802851455917 effort=33.5 velocity=21 -> lower=-0.9773843811168246 upper=0.9773843811168246 effort=53.5 velocity=11; origin xyz=-0.1805 0.047 0 rpy=0 0 0 -> xyz=-0.2305 0.055 0.01 rpy=0 0 0
- joint RL_thigh_joint: limit lower=-1.0471975512 upper=4.18879020479 effort=33.5 velocity=21 -> lower=-1.0471975511965976 upper=4.1887902047863905 effort=53.5 velocity=11; origin xyz=0 0.0838 0 rpy=0 0 0 -> xyz=0 0.1231 0 rpy=0 0 0
- joint RR_calf_joint: limit lower=-2.69653369433 upper=-0.916297857297 effort=33.5 velocity=21 -> lower=-2.8012534494508987 upper=-0.7417649320975901 effort=53.5 velocity=11; origin xyz=0 0 -0.2 rpy=0 0 0 -> xyz=0 0 -0.25 rpy=0 0 0
- joint RR_foot_fixed: origin xyz=0 0 -0.2 rpy=0 0 0 -> xyz=0.01 0 -0.2287 rpy=0 0 0
- joint RR_hip_joint: limit lower=-0.802851455917 upper=0.802851455917 effort=33.5 velocity=21 -> lower=-0.9773843811168246 upper=0.9773843811168246 effort=53.5 velocity=11; origin xyz=-0.1805 -0.047 0 rpy=0 0 0 -> xyz=-0.2305 -0.055 0.01 rpy=0 0 0
- joint RR_thigh_joint: limit lower=-1.0471975512 upper=4.18879020479 effort=33.5 velocity=21 -> lower=-1.0471975511965976 upper=4.1887902047863905 effort=53.5 velocity=11; origin xyz=0 -0.0838 0 rpy=0 0 0 -> xyz=0 -0.1231 0 rpy=0 0 0
