Commit message: 更正电机朝向

File: source/robot_lab/data/Robots/RC/DOG/urdf/DOG.urdf (robot description, URDF)
Before this commit: robot DOG, 17 links, 16 joints
Joints:
- joint FL_calf_joint: axis 0 -1 0 -> 0 1 0
- joint RR_thigh_joint: axis 0 -1 0 -> 0 1 0

Commit message: 我是秦始皇，我统一urdf

File: source/robot_lab/data/Robots/RC/DOG/urdf/DOG.urdf (robot description, URDF)
Before this commit: robot DOG, 17 links, 16 joints
Links:
- removed link FL_calf_joint
- removed link FL_feet_joint
- removed link FL_hip_joint
- removed link FL_thigh_joint
- removed link FR_calf_joint
- removed link FR_feet_joint
- removed link FR_hip_joint
- removed link FR_thigh_joint
- removed link RL_calf_joint
- removed link RL_feet_joint
- removed link RL_hip_joint
- removed link RL_thigh_joint
- removed link RR_calf_joint
- removed link RR_feet_joint
- removed link RR_hip_joint
- removed link RR_thigh_joint
- added link FL_calf_link, mass 0.1304; collision mesh filename=package://rc_description/meshes/FL_calf_joint.STL; visual mesh filename=package://rc_description/meshes/FL_calf_joint.STL
- added link FL_feet_link, mass 0.0911609; collision mesh filename=package://rc_description/meshes/FL_feet_joint.STL; visual mesh filename=package://rc_description/meshes/FL_feet_joint.STL
- added link FL_hip_link, mass 0.9754; collision mesh filename=package://rc_description/meshes/FL_hip_joint.STL; visual mesh filename=package://rc_description/meshes/FL_hip_joint.STL
- added link FL_thigh_link, mass 1.6868; collision mesh filename=package://rc_description/meshes/FL_thigh_joint.STL; visual mesh filename=package://rc_description/meshes/FL_thigh_joint.STL
- added link FR_calf_link, mass 0.1304; collision mesh filename=package://rc_description/meshes/FR_calf_joint.STL; visual mesh filename=package://rc_description/meshes/FR_calf_joint.STL
- added link FR_feet_link, mass 0.0911609; collision mesh filename=package://rc_description/meshes/FR_feet_joint.STL; visual mesh filename=package://rc_description/meshes/FR_feet_joint.STL
- added link FR_hip_link, mass 0.9754; collision mesh filename=package://rc_description/meshes/FR_hip_joint.STL; visual mesh filename=package://rc_description/meshes/FR_hip_joint.STL
- added link FR_thigh_link, mass 1.6868; collision mesh filename=package://rc_description/meshes/FR_thigh_joint.STL; visual mesh filename=package://rc_description/meshes/FR_thigh_joint.STL
- added link RL_calf_link, mass 0.1304; collision mesh filename=package://rc_description/meshes/RL_calf_joint.STL; visual mesh filename=package://rc_description/meshes/RL_calf_joint.STL
- added link RL_feet_link, mass 0.0911609; collision mesh filename=package://rc_description/meshes/RL_feet_joint.STL; visual mesh filename=package://rc_description/meshes/RL_feet_joint.STL
- added link RL_hip_link, mass 0.9754; collision mesh filename=package://rc_description/meshes/RL_hip_joint.STL; visual mesh filename=package://rc_description/meshes/RL_hip_joint.STL
- added link RL_thigh_link, mass 1.6868; collision mesh filename=package://rc_description/meshes/RL_thigh_joint.STL; visual mesh filename=package://rc_description/meshes/RL_thigh_joint.STL
- added link RR_calf_link, mass 0.1304; collision mesh filename=package://rc_description/meshes/RR_calf_joint.STL; visual mesh filename=package://rc_description/meshes/RR_calf_joint.STL
- added link RR_feet_link, mass 0.0911609; collision mesh filename=package://rc_description/meshes/RR_feet_joint.STL; visual mesh filename=package://rc_description/meshes/RR_feet_joint.STL
- added link RR_hip_link, mass 0.9754; collision mesh filename=package://rc_description/meshes/RR_hip_joint.STL; visual mesh filename=package://rc_description/meshes/RR_hip_joint.STL
- added link RR_thigh_link, mass 1.6868; collision mesh filename=package://rc_description/meshes/RR_thigh_joint.STL; visual mesh filename=package://rc_description/meshes/RR_thigh_joint.STL
- link base_link: mass 3.8805 -> 8.1152; geometry collision mesh filename=package://rc_description/meshes/base_link.STL; visual mesh filename=package://rc_description/meshes/base_link.STL
Joints:
- joint FL_calf_joint: child FL_calf_joint -> FL_calf_link; parent FL_thigh_joint -> FL_thigh_link
- joint FL_feet_joint: child FL_feet_joint -> FL_feet_link; parent FL_calf_joint -> FL_calf_link
- joint FL_hip_joint: axis -1 0 0 -> 1 0 0; child FL_hip_joint -> FL_hip_link
- joint FL_thigh_joint: child FL_thigh_joint -> FL_thigh_link; parent FL_hip_joint -> FL_hip_link
- joint FR_calf_joint: child FR_calf_joint -> FR_calf_link; parent FR_thigh_joint -> FR_thigh_link
- joint FR_feet_joint: child FR_feet_joint -> FR_feet_link; parent FR_calf_joint -> FR_calf_link
- joint FR_hip_joint: axis -1 0 0 -> 1 0 0; child FR_hip_joint -> FR_hip_link
- joint FR_thigh_joint: child FR_thigh_joint -> FR_thigh_link; parent FR_hip_joint -> FR_hip_link
- joint RL_calf_joint: child RL_calf_joint -> RL_calf_link; parent RL_thigh_joint -> RL_thigh_link
- joint RL_feet_joint: child RL_feet_joint -> RL_feet_link; parent RL_calf_joint -> RL_calf_link
- joint RL_hip_joint: child RL_hip_joint -> RL_hip_link
- joint RL_thigh_joint: child RL_thigh_joint -> RL_thigh_link; parent RL_hip_joint -> RL_hip_link
- joint RR_calf_joint: child RR_calf_joint -> RR_calf_link; parent RR_thigh_joint -> RR_thigh_link
- joint RR_feet_joint: child RR_feet_joint -> RR_feet_link; parent RR_calf_joint -> RR_calf_link
- joint RR_hip_joint: child RR_hip_joint -> RR_hip_link
- joint RR_thigh_joint: child RR_thigh_joint -> RR_thigh_link; parent RR_hip_joint -> RR_hip_link
