Commit message: 补狗脚，加入继续训练文档

File: source/robot_lab/data/Robots/RC/dog urdf/urdf/dog.urdf (robot description, URDF)
Before this commit: robot dog, 18 links, 17 joints
Links:
- removed link FL_calf_joint
- removed link FL_feet_joint
- removed link FL_hip_joint
- removed link FL_thigh_joint
- removed link FR_calf_joint
- removed link FR_feet_joint
- removed link FR_hip_joint
- removed link FR_thigh_joint
- removed link RL_calf_joint
- removed link RL_feet_joint
- removed link RL_hip_joint
- removed link RL_thigh_joint
- removed link RR_calf_joint
- removed link RR_feet_joint
- removed link RR_hip_joint
- removed link RR_thigh_joint
- removed link lidar_joint
- added link FL_calf_link, mass 0.1331; collision box size=0.1067 0.02988 0.024; visual mesh filename=package://rc_description/meshes/FL_calf_joint.STL
- added link FL_calflower1_link; collision box size=0.05 0.0258 0.025
- added link FL_calflower_link; collision box size=0.05 0.0258 0.025
- added link FL_feet_link, mass 0.0311; collision sphere radius=0.021; visual mesh filename=package://rc_description/meshes/FL_feet_joint.STL
- added link FL_hip_link, mass 0.9753; collision cylinder length=0.0631 radius=0.06275; visual mesh filename=package://rc_description/meshes/FL_hip_joint.STL
- added link FL_thigh_link, mass 1.6811; collision box size=0.25 0.065 0.085; collision cylinder length=0.0655 radius=0.054
- added link FR_calf_link, mass 0.1331; collision box size=0.1067 0.02988 0.024; visual mesh filename=package://rc_description/meshes/FR_calf_joint.STL
- added link FR_calflower1_link; collision box size=0.05 0.0258 0.025
- added link FR_calflower_link; collision box size=0.05 0.0258 0.025
- added link FR_feet_link, mass 0.0311; collision sphere radius=0.021; visual mesh filename=package://rc_description/meshes/FR_feet_joint.STL
- added link FR_hip_link, mass 0.9753; collision cylinder length=0.0631 radius=0.06275; visual mesh filename=package://rc_description/meshes/FR_hip_joint.STL
- added link FR_thigh_link, mass 1.6811; collision box size=0.25 0.065 0.085; collision cylinder length=0.0655 radius=0.054
- added link RL_calf_link, mass 0.1331; collision box size=0.1067 0.02988 0.024; visual mesh filename=package://rc_description/meshes/RL_calf_joint.STL
- added link RL_calflower1_link; collision box size=0.05 0.0258 0.025
- added link RL_calflower_link; collision box size=0.05 0.0258 0.025
- added link RL_feet_link, mass 0.0311; collision sphere radius=0.021; visual mesh filename=package://rc_description/meshes/RL_feet_joint.STL
- added link RL_hip_link, mass 0.9753; collision cylinder length=0.0631 radius=0.06275; visual mesh filename=package://rc_description/meshes/RL_hip_joint.STL
- added link RL_thigh_link, mass 1.6811; collision box size=0.25 0.065 0.085; collision cylinder length=0.0655 radius=0.054
- added link RR_calf_link, mass 0.1331; collision box size=0.1067 0.02988 0.024; visual mesh filename=package://rc_description/meshes/RR_calf_joint.STL
- added link RR_calflower1_link; collision box size=0.05 0.0258 0.025
- added link RR_calflower_link; collision box size=0.05 0.0258 0.025
- added link RR_feet_link, mass 0.0311; collision sphere radius=0.021; visual mesh filename=package://rc_description/meshes/RR_feet_joint.STL
- added link RR_hip_link, mass 0.9753; collision cylinder length=0.0631 radius=0.06275; visual mesh filename=package://rc_description/meshes/RR_hip_joint.STL
- added link RR_thigh_link, mass 1.6811; collision box size=0.25 0.065 0.085; collision cylinder length=0.0655 radius=0.054
- added link lidar_link, mass 0.2909; collision box size=0.075 0.075 0.055; visual mesh filename=package://rc_description/meshes/lidar_joint.STL
- link base_link: geometry collision box size=0.32 0.252 0.135; visual mesh filename=package://rc_description/meshes/base_link.STL
Joints:
- added joint FL_calflower1_joint: type fixed, parent FL_calflower_link, child FL_calflower1_link, origin xyz=0.03 0 -0.09 rpy=0 1.707963267948966 0, axis 0 0 0
- added joint FL_calflower_joint: type fixed, parent FL_calf_link, child FL_calflower_link, origin xyz=0 0 -0.1 rpy=0 0 0
- added joint FR_calflower1_joint: type fixed, parent FR_calflower_link, child FR_calflower1_link, origin xyz=0.03 0 -0.09 rpy=0 1.707963267948966 0, axis 0 0 0
- added joint FR_calflower_joint: type fixed, parent FR_calf_link, child FR_calflower_link, origin xyz=0 0 -0.1 rpy=0 0 0
- added joint RL_calflower1_joint: type fixed, parent RL_calflower_link, child RL_calflower1_link, origin xyz=0.03 0 -0.09 rpy=0 1.707963267948966 0, axis 0 0 0
- added joint RL_calflower_joint: type fixed, parent RL_calf_link, child RL_calflower_link, origin xyz=0 0 -0.1 rpy=0 0 0
- added joint RR_calflower1_joint: type fixed, parent RR_calflower_link, child RR_calflower1_link, origin xyz=0.03 0 -0.09 rpy=0 1.707963267948966 0, axis 0 0 0
- added joint RR_calflower_joint: type fixed, parent RR_calf_link, child RR_calflower_link, origin xyz=0 0 -0.1 rpy=0 0 0
- joint FL_calf_joint: child FL_calf_joint -> FL_calf_link; parent FL_thigh_joint -> FL_thigh_link
- joint FL_feet_joint: child FL_feet_joint -> FL_feet_link; parent FL_calf_joint -> FL_calf_link
- joint FL_hip_joint: child FL_hip_joint -> FL_hip_link
- joint FL_thigh_joint: child FL_thigh_joint -> FL_thigh_link; parent FL_hip_joint -> FL_hip_link
- joint FR_calf_joint: child FR_calf_joint -> FR_calf_link; parent FR_thigh_joint -> FR_thigh_link
- joint FR_feet_joint: child FR_feet_joint -> FR_feet_link; parent FR_calf_joint -> FR_calf_link
- joint FR_hip_joint: child FR_hip_joint -> FR_hip_link
- joint FR_thigh_joint: child FR_thigh_joint -> FR_thigh_link; parent FR_hip_joint -> FR_hip_link
- joint RL_calf_joint: child RL_calf_joint -> RL_calf_link; parent RL_thigh_joint -> RL_thigh_link
- joint RL_feet_joint: child RL_feet_joint -> RL_feet_link; parent RL_calf_joint -> RL_calf_link
- joint RL_hip_joint: child RL_hip_joint -> RL_hip_link
- joint RL_thigh_joint: child RL_thigh_joint -> RL_thigh_link; parent RL_hip_joint -> RL_hip_link
- joint RR_calf_joint: child RR_calf_joint -> RR_calf_link; parent RR_thigh_joint -> RR_thigh_link
- joint RR_feet_joint: child RR_feet_joint -> RR_feet_link; parent RR_calf_joint -> RR_calf_link
- joint RR_hip_joint: child RR_hip_joint -> RR_hip_link
- joint RR_thigh_joint: child RR_thigh_joint -> RR_thigh_link; parent RR_hip_joint -> RR_hip_link
- joint lidar_joint: child lidar_joint -> lidar_link
